Commit message: put og stuff in

File: nav2_testing/sam_bot_description/src/description/sam_bot_description.urdf (robot description, URDF)
Before this commit: robot sam_bot, 7 links, 6 joints
Links:
- removed link chassis
- added link base_link; collision box size=${base_length} ${base_width} ${base_height}; visual box size=${base_length} ${base_width} ${base_height}
Joints:
- joint base_joint: parent chassis -> base_link
- joint camera_joint: parent chassis -> base_link
- joint caster_joint: parent chassis -> base_link
- joint imu_joint: parent chassis -> base_link
- joint lidar_joint: parent chassis -> base_link
